Commit message: exercise

File: gym_panda_reach/envs/goal.urdf (robot description, URDF)
Before this commit: robot target, 1 links, 0 joints
Links:
- link baseLink: geometry collision mesh filename=objs/mug.obj; visual mesh filename=objs/mug.obj

Commit message: exercise

File: gym_panda_reach/envs/goal.urdf (robot description, URDF)
Before this commit: robot target, 1 links, 0 joints
Links:
- link baseLink: geometry collision mesh filename=objects/007_tuna_fish_can/google_16k/textured.obj; visual mesh filename=objects/007_tuna_fish_can/google_16k/textured.obj

Commit message: exercise

File: gym_panda_reach/envs/goal.urdf (robot description, URDF)
Before this commit: robot target, 1 links, 0 joints
Links:
- link baseLink: geometry collision mesh filename=objects/mug.obj; visual mesh filename=objects/mug.obj
